File: pcb/ecp5u85-bse-usb_io-tester.kicad_sch (KiCad schematic)
At the start: 95 parts, among them J1 BTE-040-02-L-D-A, J2 USB_B_Mini, J3 BTE-040-02-L-D-A, J4 Conn_02x03_Odd_Even, J5 Conn_02x10_Odd_Even, SW1 SW_Push, U1 74HCT4067PW,118, U10 74HCT4067PW,118, U11 74HCT4067PW,118, U12 FT232RL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

Commit message: Added fabrication files for Rev. A
- SMD mounts are specified in smd-mount as CSV and in gerber as
  *-pnp_top.gbr and *-pnp-bottom.gbr
- Fabrication information containing component reference designators and
  values are in gerber/*_Fab.gbr
- The bill of materials is in bom folder. It can be exported to CSV in
  the browser application.
Parts:
- removed L1: L, Inductor_SMD:L_1206_3216Metric, symbol Device:L
- added FB2: FBMH3216HM221NTV, Inductor_SMD:L_1206_3216Metric, symbol Device:FerriteBead
- C15: value 100uF -> T498X107K016ATE075; footprint Capacitor_Tantalum_SMD:CP_EIA-6032-28_Kemet-C -> Capacitor_Tantalum_SMD:CP_EIA-7343-20_Kemet-V
- D1, D2, D3, D5, D6: value LED -> LTST-C191KGKT
- FB1: value FerriteBead -> MH1608-601Y
- J2: value USB_B_Mini -> 65100516121; footprint Connector_USB:USB_Mini-B_Lumberg_2486_01_Horizontal -> Connector_USB:USB_Mini-B_Wuerth_65100516121_Horizontal
- J4: value Conn_02x03_Odd_Even -> 67996-206HLF
- J5: value Conn_02x10_Odd_Even -> 67996-420HLF
- RN1, RN10, RN11, RN12, RN13, RN14, RN15, RN16, RN2, RN3, RN4, RN5, RN6, RN7, RN8, RN9: value 4609X-AP1-103LF -> 745X101103JP
- SW1: value SW_Push -> B3F-1002
- U13: value OSCILLATOR_EN -> O 32,0-JT32C-A-K-3,3-LF
Connections:
- net +5V: now also FB2.2
- net VBUS: now also FB2.1
